File: hardware/qtpy_midibff_disp.brd (EAGLE design)
At the start: 54 x 22 mm, 9 parts, among them J1 SJ-3523-SMT, J2 SJ-3523-SMT, U1 ADAFRUIT_QTPYM0, U2 6N137

Commit message: sigh trs-a/b will kill me
Parts:
- added C1: (no value), rcl:C025-025X050
Connections:
- removed net M_IN: J2.2, R3.2
- removed net M_OUT: J1.2, R1.1
- new net N$3: J2.2, U2.3
- new net N$5: J1.2, R2.1
- net +3V3: now also C1.1
- net GND: now also C1.2
- net N$1: now also R1.1; no longer R2.1
- net N$4: now also R3.2; no longer U2.3
Routing:
- net M_IN: track 9.49 -> 0.00 mm
- net N$4: track 14.8 -> 21.9 mm
- net N$5: track 0.00 -> 6.51 mm, vias 0 -> 1
- net N$3: track 0.00 -> 6.40 mm
- net M_OUT: track 5.47 -> 0.00 mm
- net N$1: track 14.7 -> 16.4 mm
Other:
- board text added: "qtpy_midibff_disp_5Aug2022"
- board text removed: "qtpy_midibff_disp_22Jul2022"
