File: schematics/midi_bff/midi_bff.kicad_sch (KiCad schematic)
At the start: 18 parts, among them CN1 DIN-504, CN2 DIN-504, J1 PJ-320A-4P DIP, J2 PJ-320A-4P DIP, J3 OLED-128x32, U3 H11L1

Commit message: add LED status to all Arduino sketches
Parts:
- renumbered C28 to C1
Changed lines of the file:
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@@
 		(in_pos_files yes)
 		(dnp no)
-		(property "Reference" "C28"
+		(property "Reference" "C1"
 			(at 127 23.876 0)
 			(show_name no)
@@
 			(project "midi_bff"
 				(path "/c90acee2-2190-4772-922f-6881161c54a7"
-					(reference "C28")
+					(reference "C1")
 					(unit 1)
 				)
