File: schematics/midi_bff/midi_bff.kicad_pcb (KiCad board)
At the start: 2 copper layers, 63.5 x 44.4 mm, 18 parts, among them CN1 DIN-504, CN2 DIN-504, J1 PJ-320A-4P DIP, J2 PJ-320A-4P DIP, J3 OLED-128x32, U3 H11L1

Commit message: add led blinking on midi
Parts:
- renumbered C28 to C1
Changed lines of the file:
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@@
 		(descr "C, Disc series, Radial, pin pitch=2.50mm, diameter*width=3.0*1.6mm^2, Capacitor, http://www.vishay.com/docs/45233/krseries.pdf")
 		(tags "C Disc series Radial pin pitch 2.50mm diameter 3.0mm width 1.6mm Capacitor")
-		(property "Reference" "C28"
+		(property "Reference" "C1"
 			(at 5.08 0 0)
 			(layer "F.SilkS")
